Commit message: trying to add a camera

File: franka_description/robots/hand.xacro (robot description, xacro)
@@ -82,4 +82,62 @@
       <limit effort="20" lower="0.0" upper="0.04" velocity="0.2"/>
     </joint>
+    <!-- attach a camera frame -->
+    <link name="${ns}_hand_camera">
+      <visual>
+        <origin xyz="0 0 0" rpy="0 0 0" />
+        <geometry>
+          <box size="0.1 0.03 0.01" />
+        </geometry>
+        <material name="cam_color">
+          <color rgba="0. 1. 0. 0.3" />
+        </material>
+      </visual>
+      <inertial>
+        <origin xyz="0 0 0" rpy="0 0 0" />
+        <mass value="0.01" />
+        <inertia ixx="0.1" ixy="0.0" ixz="0.0" iyy="0.1" iyz="0.0" izz="0.1" />
+      </inertial>
+    </link>
+    <joint name="${ns}_camera_joint" type="fixed">
+      <parent link="${ns}_hand" />
+      <child link="${ns}_hand_camera" />
+      <origin xyz="0.1 0 0" rpy="0 0 ${pi/2}" />
+    </joint>
+    <gazebo reference="${ns}_camera_link">
+      <sensor type="camera" name="${ns}_camera">
+        <update_rate>10.0</update_rate>
+        <camera name="camera">
+          <horizontal_fov>1.396</horizontal_fov>
+          <image>
+            <width>640</width>
+            <height>480</height>
+            <format>R8G8B8</format>
+          </image>
+          <clip>
+            <near>0.02</near>
+            <far>30</far>
+          </clip>
+          <noise>
+            <type>gaussian</type>
+            <mean>0.0</mean>
+            <stddev>0.007</stddev>
+          </noise>
+        </camera>
+        <plugin name="camera_controller" filename="libgazebo_ros_camera.so">
+          <alwaysOn>true</alwaysOn>
+          <updateRate>0.0</updateRate>
+          <cameraName>panda/camera</cameraName>
+          <imageTopicName>image_raw</imageTopicName>
+          <cameraInfoTopicName>camera_info</cameraInfoTopicName>
+          <frameName>camera_link</frameName>
+          <hackBaseline>0.07</hackBaseline>
+          <distortionK1>0.0</distortionK1>
+          <distortionK2>0.0</distortionK2>
+          <distortionK3>0.0</distortionK3>
+          <distortionT1>0.0</distortionT1>
+          <distortionT2>0.0</distortionT2>
+        </plugin>
+      </sensor>
+    </gazebo>
   </xacro:macro>
 </robot>

Commit message: added calibration target, fixed camera transforms

File: franka_description/robots/hand.xacro (robot description, xacro)
@@ -83,9 +83,9 @@
     </joint>
     <!-- attach a camera frame -->
-    <link name="${ns}_hand_camera">
+    <link name="${ns}_camera_link">
       <visual>
         <origin xyz="0 0 0" rpy="0 0 0" />
         <geometry>
-          <box size="0.1 0.03 0.01" />
+          <box size="0.01 0.1 0.03" />
         </geometry>
         <material name="cam_color">
@@ -99,8 +99,14 @@
       </inertial>
     </link>
+    <link name="${ns}_camera_optical_frame" />
     <joint name="${ns}_camera_joint" type="fixed">
       <parent link="${ns}_hand" />
-      <child link="${ns}_hand_camera" />
-      <origin xyz="0.1 0 0" rpy="0 0 ${pi/2}" />
+      <child link="${ns}_camera_link" />
+      <origin xyz="0.1 0 0" rpy="0 ${-pi/2} ${pi}" />
+    </joint>
+    <joint name="${ns}_camera_optical_joint" type="fixed">
+      <parent link="${ns}_camera_link" />
+      <child link="${ns}_camera_optical_frame" />
+      <origin xyz="0 0 0" rpy="${-pi/2} 0 ${-pi/2}" />
     </joint>
     <gazebo reference="${ns}_camera_link">
@@ -127,8 +133,8 @@
           <alwaysOn>true</alwaysOn>
           <updateRate>0.0</updateRate>
-          <cameraName>panda/camera</cameraName>
+          <cameraName>${ns}/camera</cameraName>
           <imageTopicName>image_raw</imageTopicName>
           <cameraInfoTopicName>camera_info</cameraInfoTopicName>
-          <frameName>camera_link</frameName>
+          <frameName>${ns}_camera_optical_frame</frameName>
           <hackBaseline>0.07</hackBaseline>
           <distortionK1>0.0</distortionK1>

File: franka_description/robots/panda_arm_hand.urdf.xacro (robot description, xacro)
@@ -13,3 +13,7 @@
   <xacro:panda_control arm_id="panda" load_hand="true" />
   <!-- end for simulation -->
+  <!-- calibration target -->
+  <xacro:include filename="$(find franka_description)/robots/calibration_target.xacro" />
+  <xacro:calibration_target  xyz="2 0 1" rpy="0 0 0" connected_to="world" />
+  <!-- end calibration target -->
 </robot>

Commit message: hide real calibration

File: franka_description/robots/hand.xacro (robot description, xacro)
@@ -99,5 +99,4 @@
       </inertial>
     </link>
-    <link name="${ns}_camera_optical_frame" />
     <joint name="${ns}_camera_joint" type="fixed">
       <parent link="${ns}_hand" />
@@ -105,4 +104,6 @@
       <origin xyz="0.1 0 0" rpy="0 ${-pi/2} ${pi}" />
     </joint>
+    <!--
+    <link name="${ns}_camera_optical_frame" />
     <joint name="${ns}_camera_optical_joint" type="fixed">
       <parent link="${ns}_camera_link" />
@@ -110,4 +111,5 @@
       <origin xyz="0 0 0" rpy="${-pi/2} 0 ${-pi/2}" />
     </joint>
+    -->
     <gazebo reference="${ns}_camera_link">
       <sensor type="camera" name="${ns}_camera">
