Commit message: fix rviz malformed url error

File: franka_description/robots/calibration_target.xacro (robot description, xacro)
@@ -13,5 +13,5 @@
         <origin xyz="0 0 0" rpy="0 1.57 0" />
         <geometry>
-          <mesh filename="$(find franka_description)/meshes/visual/calibration_target.dae"/>
+          <mesh filename="file://$(find franka_description)/meshes/visual/calibration_target.dae"/>
         </geometry>
       </visual>
@@ -19,5 +19,5 @@
         <origin xyz="0 0 0" rpy="0 1.57 0" />
         <geometry>
-          <mesh filename="$(find franka_description)/meshes/visual/calibration_target.dae"/>
+          <mesh filename="file://$(find franka_description)/meshes/visual/calibration_target.dae"/>
         </geometry>
       </collision>

Commit message: ChArUco target

File: franka_description/robots/calibration_target.xacro (robot description, xacro)
@@ -13,5 +13,5 @@
         <origin xyz="0 0 0" rpy="0 1.57 0" />
         <geometry>
-          <mesh filename="file://$(find franka_description)/meshes/visual/calibration_target.dae"/>
+          <mesh filename="file://$(find franka_description)/meshes/visual/charuco_calibration_target.dae"/>
         </geometry>
       </visual>
@@ -19,5 +19,5 @@
         <origin xyz="0 0 0" rpy="0 1.57 0" />
         <geometry>
-          <mesh filename="file://$(find franka_description)/meshes/visual/calibration_target.dae"/>
+          <mesh filename="file://$(find franka_description)/meshes/visual/charuco_calibration_target.dae"/>
         </geometry>
       </collision>
